Commit message: Update URDF.
Signed-off-by: James Goppert <james.goppert@gmail.com>

File: rdd2_description/urdf/rdd2.urdf (robot description, URDF)
Before this commit: robot rdd2, 5 links, 4 joints
Joints:
- joint base_joint: origin xyz=0.0 0.0 0.0 rpy=0 0 0 -> xyz=0.0 0.0 -0.23 rpy=0 0 0
- joint camera_joint: origin xyz=.173 0 .145 rpy=0 0 0 -> xyz=.13 0 -0.05 rpy=0 0 0
- joint lidar_joint: origin xyz=0 0 0.191 rpy=0 0 0 -> xyz=0 0 0.08 rpy=0 0 0
